Commit message: friction_changed

File: urdf/abb_gripper_macro.xacro (robot description, xacro)
@@ -44,6 +44,5 @@
       <child link="${gripper_prefix}ABB_Gripper_Finger_1" />
       <axis xyz="-1 0 0" />
-      <dynamics damping="0.5" friction="0.0"/>
-      <limit lower="0.0" upper="0.0135" effort="100.0" velocity="1.0"/>
+      <limit lower="0.0" upper="0.0135" effort="200.0" velocity="1.0"/>
     </joint>
     <link name="${gripper_prefix}ABB_Gripper_Finger_2">
@@ -65,10 +64,52 @@
       <child link="${gripper_prefix}ABB_Gripper_Finger_2" />
       <axis xyz="1 0 0" />
-      <dynamics damping="0.5" friction="0.0"/>
-      <limit lower="0.0" upper="0.0135" effort="100.0" velocity="1.0"/>
+      <limit lower="0.0" upper="0.0135" effort="200.0" velocity="1.0"/>
     </joint>
-    <!-- ================= ROS2 CONTROL & GAZEBO PLUGIN CONSOLIDATED ================= -->
-    <!-- These blocks have been removed from this file and must be placed
-         in the top-level dual_arms Xacro file. -->
+    <gazebo reference="${gripper_prefix}ABB_Gripper_Finger_1">
+      <surface>
+        <friction>
+          <torsional>
+            <ode/>
+          </torsional>
+          <ode>
+            <mu>100</mu>
+            <mu2>100</mu2>
+            <slip1>0.0</slip1>
+            <slip2>0.0</slip2>
+          </ode>
+        </friction>
+        <contact>
+          <ode>
+            <max_vel>0.0</max_vel>
+            <min_depth>0.001</min_depth>
+            <kp>100000</kp>
+            <kd>10</kd>
+          </ode>
+        </contact>
+      </surface>
+    </gazebo>
+    <gazebo reference="${gripper_prefix}ABB_Gripper_Finger_2">
+      <surface>
+        <friction>
+          <torsional>
+            <ode/>
+          </torsional>
+          <ode>
+            <mu>100</mu>
+            <mu2>100</mu2>
+            <slip1>0.0</slip1>
+            <slip2>0.0</slip2>
+          </ode>
+        </friction>
+        <contact>
+          <ode>
+            <max_vel>0.0</max_vel>
+            <min_depth>0.001</min_depth>
+            <kp>100000</kp>
+            <kd>10</kd>
+          </ode>
+        </contact>
+      </surface>
+    </gazebo>
   </xacro:macro>
 </robot>

Commit message: gripping_physiscs_last_version

File: urdf/abb_gripper_macro.xacro (robot description, xacro)
@@ -37,5 +37,8 @@
       </visual>
       <collision>
-        <geometry><mesh filename="package://abb_gripper_urdf/meshes/ABB_Gripper_Finger_1.STL" /></geometry>
+        <origin xyz="-0.0123 0.17 -0.0015" rpy="0 0 0" />
+        <geometry>
+          <box size="0.013 0.04 0.018" />
+        </geometry>
       </collision>
     </link>
@@ -44,5 +47,5 @@
       <child link="${gripper_prefix}ABB_Gripper_Finger_1" />
       <axis xyz="-1 0 0" />
-      <limit lower="0.0" upper="0.0135" effort="200.0" velocity="1.0"/>
+      <limit lower="0.0" upper="0.0135" effort="20.0" velocity="1.0"/>
     </joint>
     <link name="${gripper_prefix}ABB_Gripper_Finger_2">
@@ -57,5 +60,8 @@
       </visual>
       <collision>
-        <geometry><mesh filename="package://abb_gripper_urdf/meshes/ABB_Gripper_Finger_2.STL" /></geometry>
+        <origin xyz="0.0122 0.17 -0.0015" rpy="0 0 0" />
+        <geometry>
+          <box size="0.013 0.04 0.018" />
+        </geometry>
       </collision>
     </link>
@@ -64,5 +70,5 @@
       <child link="${gripper_prefix}ABB_Gripper_Finger_2" />
       <axis xyz="1 0 0" />
-      <limit lower="0.0" upper="0.0135" effort="200.0" velocity="1.0"/>
+      <limit lower="0.0" upper="0.0135" effort="20.0" velocity="1.0"/>
     </joint>
     <gazebo reference="${gripper_prefix}ABB_Gripper_Finger_1">
@@ -70,9 +76,13 @@
         <friction>
           <torsional>
-            <ode/>
+            <ode>
+              <coefficient>100.0</coefficient>
+              <use_patch_radius>true</use_patch_radius>
+              <patch_radius>0.015</patch_radius>
+            </ode>
           </torsional>
           <ode>
-            <mu>100</mu>
-            <mu2>100</mu2>
+            <mu>100.0</mu>
+            <mu2>100.0</mu2>
             <slip1>0.0</slip1>
             <slip2>0.0</slip2>
@@ -83,6 +93,6 @@
             <max_vel>0.0</max_vel>
             <min_depth>0.001</min_depth>
-            <kp>100000</kp>
-            <kd>10</kd>
+            <kp>1000000.0</kp>
+            <kd>1.0</kd>
           </ode>
         </contact>
@@ -93,9 +103,13 @@
         <friction>
           <torsional>
-            <ode/>
+            <ode>
+              <coefficient>100.0</coefficient>
+              <use_patch_radius>true</use_patch_radius>
+              <patch_radius>0.015</patch_radius>
+            </ode>
           </torsional>
           <ode>
-            <mu>100</mu>
-            <mu2>100</mu2>
+            <mu>100.0</mu>
+            <mu2>100.0</mu2>
             <slip1>0.0</slip1>
             <slip2>0.0</slip2>
@@ -106,6 +120,6 @@
             <max_vel>0.0</max_vel>
             <min_depth>0.001</min_depth>
-            <kp>100000</kp>
-            <kd>10</kd>
+            <kp>1000000.0</kp>
+            <kd>1.0</kd>
           </ode>
         </contact>

Commit message: gripper meya meya

File: urdf/abb_gripper_macro.xacro (robot description, xacro)
@@ -47,5 +47,5 @@
       <child link="${gripper_prefix}ABB_Gripper_Finger_1" />
       <axis xyz="-1 0 0" />
-      <limit lower="0.0001" upper="0.0135" effort="20.0" velocity="1.0"/>
+      <limit lower="0.001" upper="0.014" effort="5.0" velocity="1.0"/>
     </joint>
     <link name="${gripper_prefix}ABB_Gripper_Finger_2">
@@ -70,5 +70,5 @@
       <child link="${gripper_prefix}ABB_Gripper_Finger_2" />
       <axis xyz="1 0 0" />
-      <limit lower="0.0001" upper="0.0135" effort="20.0" velocity="1.0"/>
+      <limit lower="0.001" upper="0.014" effort="5.0" velocity="1.0"/>
     </joint>
     <gazebo reference="${gripper_prefix}ABB_Gripper_Finger_1">
